Commit message: got imu working

File: ros2_gazebo_sim/urdf/model.urdf (robot description, URDF)
Before this commit: robot virtual_robot, 13 links, 12 joints
Links:
- removed link car_1_base_link
- removed link car_1_camera_link
- removed link car_1_chassis
- removed link car_1_chassis_inertia
- removed link car_1_laser
- removed link car_1_left_front_wheel
- removed link car_1_left_rear_wheel
- removed link car_1_left_steering_hinge
- removed link car_1_link
- removed link car_1_right_front_wheel
- removed link car_1_right_link
- removed link car_1_right_rear_wheel
- removed link car_1_right_steering_hinge
- added link base_link
- added link camera_link, mass 1e-5
- added link chassis; collision mesh filename=model://urdf/meshes/chassis.stl scale=0.000990 0.0009375 0.0009375; visual mesh filename=model://urdf/meshes/chassis.stl scale=0.000990 0.0009375 0.0009375
- added link chassis_inertia, mass 4.0
- added link imu_link, mass 0.1; collision box size=0.1 0.1 0.1; visual box size=0.1 0.1 0.1
- added link laser, mass 0.130; collision box size=0.1 0.1 0.1; visual mesh filename=model://urdf/meshes/hokuyo.stl
- added link left_front_wheel, mass 0.34055; collision cylinder length=0.045 radius=0.05; visual mesh filename=model://urdf/meshes/left_wheel.stl
- added link left_rear_wheel, mass 0.34055; collision cylinder length=0.045 radius=0.05; visual mesh filename=model://urdf/meshes/left_wheel.stl
- added link left_steering_hinge, mass 0.100; visual mesh filename=model://urdf/meshes/hinge.stl
- added link link, mass 1e-5; collision box size=0.033 0.175 0.030; visual box size=0.033 0.175 0.030
- added link right_front_wheel, mass 0.34055; collision cylinder length=0.045 radius=0.05; visual mesh filename=model://urdf/meshes/right_wheel.stl
- added link right_link, mass 1e-5
- added link right_rear_wheel, mass 0.34055; collision cylinder length=0.045 radius=0.05; visual mesh filename=model://urdf/meshes/right_wheel.stl
- added link right_steering_hinge, mass 0.100; visual mesh filename=model://urdf/meshes/hinge.stl
Joints:
- removed joint car_1_base_link_joint
- removed joint car_1_chassis_inertia_joint
- removed joint car_1_hokuyo_joint
- removed joint car_1_joint
- removed joint car_1_left_front_wheel_joint
- removed joint car_1_left_joint
- removed joint car_1_left_rear_wheel_joint
- removed joint car_1_left_steering_hinge_joint
- removed joint car_1_right_front_wheel_joint
- removed joint car_1_right_joint
- removed joint car_1_right_rear_wheel_joint
- removed joint car_1_right_steering_hinge_joint
- added joint base_link_joint: type fixed, parent base_link, child chassis, origin xyz=0 0 0.05 rpy=0 0 0
- added joint chassis_inertia_joint: type fixed, parent chassis, child chassis_inertia, origin xyz=0 0 0 rpy=0 0 0
- added joint hokuyo_joint: type fixed, parent chassis, child laser, origin xyz=0.125 0.0 0.173 rpy=0 0 0, axis 0 0 1
- added joint imu_joint: type fixed, parent base_link, child imu_link, origin xyz=0 0 0.01
- added joint joint: type fixed, parent chassis, child link, origin xyz=0.390 0 0.025 rpy=0 0 0, axis 0 0 1
- added joint left_front_wheel_joint: type continuous, parent left_steering_hinge, child left_front_wheel, origin xyz=0 0 0 rpy=1.5708 0 0, axis 0 0 -1, limit effort=10 velocity=100
- added joint left_joint: type fixed, parent link, child camera_link, origin xyz=-2.5 0 1.75 rpy=0 .57 0, axis 0 0 1
- added joint left_rear_wheel_joint: type continuous, parent chassis, child left_rear_wheel, origin xyz=0 0.1 0 rpy=1.5708 0 0, axis 0 0 -1, limit effort=10 velocity=100
- added joint left_steering_hinge_joint: type revolute, parent chassis, child left_steering_hinge, origin xyz=0.325 0.1 0 rpy=0 1.5708 0, axis -1 0 0, limit lower=-1.0 upper=1.0 effort=10 velocity=100
- added joint right_front_wheel_joint: type continuous, parent right_steering_hinge, child right_front_wheel, origin xyz=0 0 0 rpy=1.5708 0 0, axis 0 0 -1, limit effort=10 velocity=100
- added joint right_joint: type fixed, parent link, child right_link, origin xyz=0 -0.06 0.025 rpy=0 0 0, axis 0 0 1
- added joint right_rear_wheel_joint: type continuous, parent chassis, child right_rear_wheel, origin xyz=0 -0.1 0 rpy=1.5708 0 0, axis 0 0 -1, limit effort=10 velocity=100
- added joint right_steering_hinge_joint: type revolute, parent chassis, child right_steering_hinge, origin xyz=0.325 -0.1 0 rpy=0 1.5708 0, axis -1 0 0, limit lower=-1.0 upper=1.0 effort=10 velocity=100
