Commit message: updated README to reflect that our simulator is now a ROS package

File: ros2_gazebo_sim/urdf/macros.xacro (robot description, xacro)
@@ -44,5 +44,5 @@
     <origin xyz="0.46 -0.135 -0.180" rpy="1.57 0 3.14" />
     <geometry>
-      <mesh filename="/sim_ws/src/urdf/meshes/chassis.stl" scale="0.000990 0.0009375 0.0009375"/>
+      <mesh filename="package://ros2_gazebo_sim/urdf/meshes/chassis.stl" scale="0.000990 0.0009375 0.0009375"/>
     </geometry>
   </xacro:macro>
@@ -50,5 +50,5 @@
     <origin xyz="0 0 0" rpy="0 0 0" />
     <geometry>
-      <mesh filename="/sim_ws/src/urdf/meshes/left_wheel.stl" />
+      <mesh filename="package://ros2_gazebo_sim/urdf/meshes/left_wheel.stl" />
     </geometry>
   </xacro:macro>
@@ -56,5 +56,5 @@
     <origin xyz="0 0 0" rpy="0 0 0" />
     <geometry>
-      <mesh filename="/sim_ws/src/urdf/meshes/right_wheel.stl" />
+      <mesh filename="package://ros2_gazebo_sim/urdf/meshes/right_wheel.stl" />
     </geometry>
   </xacro:macro>
@@ -62,5 +62,5 @@
     <origin xyz="0 0 0" rpy="0 0 0" />
     <geometry>
-      <mesh filename="/sim_ws/src/urdf/meshes/left_wheel.stl" />
+      <mesh filename="package://ros2_gazebo_sim/urdf/meshes/left_wheel.stl" />
     </geometry>
   </xacro:macro>
@@ -68,5 +68,5 @@
     <origin xyz="0 0 0" rpy="0 0 0" />
     <geometry>
-      <mesh filename="/sim_ws/src/urdf/meshes/right_wheel.stl" />
+      <mesh filename="package://ros2_gazebo_sim/urdf/meshes/right_wheel.stl" />
     </geometry>
   </xacro:macro>
@@ -74,5 +74,5 @@
     <origin xyz="0 0 0" rpy="0 0 0" />
     <geometry>
-      <mesh filename="/sim_ws/src/urdf/meshes/hinge.stl" />
+      <mesh filename="package://ros2_gazebo_sim/urdf/meshes/hinge.stl" />
     </geometry>
   </xacro:macro>
@@ -80,5 +80,5 @@
     <origin xyz="0 0 0" rpy="0 0 0" />
     <geometry>
-      <mesh filename="/sim_ws/src/urdf/meshes/hinge.stl" />
+      <mesh filename="package://ros2_gazebo_sim/urdf/meshes/hinge.stl" />
     </geometry>
   </xacro:macro>
@@ -99,11 +99,16 @@
     <transmission name="${name}_transmission" type="SimpleTransmission">
       <type>transmission_interface/SimpleTransmission</type>
-      <joint name="${name}_joint">
-        <hardwareInterface>hardware_interface/EffortJointInterface</hardwareInterface>
-      </joint>
-      <actuator name="${name}_motor">
-        <hardwareInterface>hardware_interface/EffortJointInterface</hardwareInterface>
-        <mechanicalReduction>1</mechanicalReduction>
-      </actuator>
+      <ros2_control name="GazeboSimSystem" type="system">
+        <hardware>
+          <plugin>gz_ros2_control/GazeboSimSystem</plugin>
+        </hardware>
+        <joint name="${name}_joint">
+          <hardwareInterface>hardware_interface/EffortJointInterface</hardwareInterface>
+        </joint>
+        <actuator name="${name}_motor">
+          <hardwareInterface>hardware_interface/EffortJointInterface</hardwareInterface>
+          <mechanicalReduction>1</mechanicalReduction>
+        </actuator>
+      </ros2_control>
     </transmission>
   </xacro:macro>
@@ -111,11 +116,16 @@
     <transmission name="${name}_transmission" type="SimpleTransmission">
       <type>transmission_interface/SimpleTransmission</type>
-      <joint name="${name}_joint">
-        <hardwareInterface>hardware_interface/EffortJointInterface</hardwareInterface>
-      </joint>
-      <actuator name="${name}_motor">
-        <hardwareInterface>hardware_interface/EffortJointInterface</hardwareInterface>
-        <mechanicalReduction>1</mechanicalReduction>
-      </actuator>
+      <ros2_control name="GazeboSimSystem" type="system">
+        <hardware>
+          <plugin>gz_ros2_control/GazeboSimSystem</plugin>
+        </hardware>
+        <joint name="${name}_joint">
+          <hardwareInterface>hardware_interface/EffortJointInterface</hardwareInterface>
+        </joint>
+        <actuator name="${name}_motor">
+          <hardwareInterface>hardware_interface/EffortJointInterface</hardwareInterface>
+          <mechanicalReduction>1</mechanicalReduction>
+        </actuator>
+      </ros2_control>
     </transmission>
   </xacro:macro>
@@ -280,5 +290,5 @@
       <origin xyz="0 0 -0.018" rpy="0 0 0"/>
       <geometry>
-        <mesh filename="/sim_ws/src/urdf/meshes/hokuyo.stl"/>
+        <mesh filename="package://ros2_gazebo_sim/urdf/meshes/hokuyo.stl"/>
         <material name="grey" />
       </geometry>
@@ -387,11 +397,10 @@
   </gazebo>
   <!-- Gazebo plugins -->
-  <!-- <gazebo>
-    <plugin name="gazebo_ros_control" filename="libgazebo_ros_control.so">
-      <robotNamespace>/$(arg robot_name)</robotNamespace>
-      <robotSimType>gazebo_ros_control/DefaultRobotHWSim</robotSimType>
+  <gazebo>
+    <plugin filename="libgz_ros2_control-system.so" name="gz_ros2_control::GazeboSimROS2ControlPlugin">
+      <parameters>$(find gz_ros2_control_demos)/config/control.yaml</parameters>
     </plugin>
   </gazebo>
-  Odometry (cheap hack)
+  <!-- Odometry (cheap hack) -->
   <gazebo>
     <plugin name="p3d_base_controller" filename="libgazebo_ros_p3d.so">
@@ -405,5 +414,5 @@
       <rpyOffsets>0 0 0</rpyOffsets>
     </plugin>
-  </gazebo> -->
+  </gazebo>
   <!-- hokuyo -->
   <xacro:unless value="$(optenv DISABLE_GAZEBO_LASER false)">
@@ -433,10 +442,8 @@
           </noise>
         </ray>
-        <!-- <plugin name="hokuyo_controller" filename="libgazebo_ros_laser.so">
+        <plugin name="hokuyo_controller" filename="libgazebo_ros_laser.so">
           <topicName>/$(arg robot_name)/scan</topicName>
           <frameName>$(arg robot_name)_laser</frameName>
-        </plugin> -->
-        <topic>scan</topic>
-        <gz_frame_id>$(arg robot_name)_laser</gz_frame_id>
+        </plugin>
       </sensor>
     </gazebo>
@@ -448,8 +455,5 @@
         <update_rate>30.0</update_rate>
         <!-- math.atan(320 / 687.8065795898438) * 2 -->
-        <gz_frame_id>$(arg robot_name)_camera_link</gz_frame_id>
-        <topic>camera/image_raw</topic>
         <camera name="front_camera">
-          <camera_info_topic>camera/camera_info</camera_info_topic>
           <!-- horizontal_fov>0.8709216071359963</horizontal_fov -->
           <horizontal_fov>1.74</horizontal_fov>
@@ -469,11 +473,12 @@
           </noise>
         </camera>
-        <!-- <plugin name="camera_controller" filename="libgazebo_ros_camera.so">
+        <plugin name="camera_controller" filename="libgazebo_ros_camera.so">
           <alwaysOn>true</alwaysOn>
           <updateRate>30.0</updateRate>
           <cameraName>/$(arg robot_name)/camera</cameraName>
           <imageTopicName>image</imageTopicName>
+          <cameraInfoTopicName>rgb/camera_info</cameraInfoTopicName>
           <frameName>$(arg robot_name)_camera_link</frameName>
-          <hackBaseline>0</hackBaseline>set this to 0.12 for the second camera
+          <hackBaseline>0</hackBaseline><!-- set this to 0.12 for the second camera -->
           <distortionK1>0.0</distortionK1>
           <distortionK2>0.0</distortionK2>
@@ -481,5 +486,5 @@
           <distortionT1>0.0</distortionT1>
           <distortionT2>0.0</distortionT2>
-        </plugin> -->
+        </plugin>
       </sensor>
     </gazebo>

Commit message: car appears successfully with custom package

File: ros2_gazebo_sim/urdf/macros.xacro (robot description, xacro)
@@ -44,5 +44,5 @@
     <origin xyz="0.46 -0.135 -0.180" rpy="1.57 0 3.14" />
     <geometry>
-      <mesh filename="package://ros2_gazebo_sim/urdf/meshes/chassis.stl" scale="0.000990 0.0009375 0.0009375"/>
+      <mesh filename="model://urdf/meshes/chassis.stl" scale="0.000990 0.0009375 0.0009375"/>
     </geometry>
   </xacro:macro>
@@ -50,5 +50,5 @@
     <origin xyz="0 0 0" rpy="0 0 0" />
     <geometry>
-      <mesh filename="package://ros2_gazebo_sim/urdf/meshes/left_wheel.stl" />
+      <mesh filename="model://urdf/meshes/left_wheel.stl" />
     </geometry>
   </xacro:macro>
@@ -56,5 +56,5 @@
     <origin xyz="0 0 0" rpy="0 0 0" />
     <geometry>
-      <mesh filename="package://ros2_gazebo_sim/urdf/meshes/right_wheel.stl" />
+      <mesh filename="model://urdf/meshes/right_wheel.stl" />
     </geometry>
   </xacro:macro>
@@ -62,5 +62,5 @@
     <origin xyz="0 0 0" rpy="0 0 0" />
     <geometry>
-      <mesh filename="package://ros2_gazebo_sim/urdf/meshes/left_wheel.stl" />
+      <mesh filename="model://urdf/meshes/left_wheel.stl" />
     </geometry>
   </xacro:macro>
@@ -68,5 +68,5 @@
     <origin xyz="0 0 0" rpy="0 0 0" />
     <geometry>
-      <mesh filename="package://ros2_gazebo_sim/urdf/meshes/right_wheel.stl" />
+      <mesh filename="model://urdf/meshes/right_wheel.stl" />
     </geometry>
   </xacro:macro>
@@ -74,5 +74,5 @@
     <origin xyz="0 0 0" rpy="0 0 0" />
     <geometry>
-      <mesh filename="package://ros2_gazebo_sim/urdf/meshes/hinge.stl" />
+      <mesh filename="model://urdf/meshes/hinge.stl" />
     </geometry>
   </xacro:macro>
@@ -80,5 +80,5 @@
     <origin xyz="0 0 0" rpy="0 0 0" />
     <geometry>
-      <mesh filename="package://ros2_gazebo_sim/urdf/meshes/hinge.stl" />
+      <mesh filename="model://urdf/meshes/hinge.stl" />
     </geometry>
   </xacro:macro>
@@ -97,37 +97,34 @@
   <!-- transmission macros -->
   <xacro:macro name="wheel_transmission" params="name">
+    <ros2_control name="${name}_transmission" type="actuator">
+      <hardware>
+        <plugin>gz_ros2_control/GazeboSimSystem</plugin>
+      </hardware>
+      <joint name="${name}_joint">
+      </joint>
+    </ros2_control>
+    <!-- <transmission name="${name}_transmission" type="SimpleTransmission">
+      <type>transmission_interface/SimpleTransmission</type>
+      <joint name="${name}_joint">
+        <hardwareInterface>hardware_interface/EffortJointInterface</hardwareInterface>
+      </joint>
+      <actuator name="${name}_motor">
+        <hardwareInterface>hardware_interface/EffortJointInterface</hardwareInterface>
+        <mechanicalReduction>1</mechanicalReduction>
+      </actuator>
+    </transmission> -->
+  </xacro:macro>
+  <!-- <xacro:macro name="steering_hinge_transmission" params="name">
     <transmission name="${name}_transmission" type="SimpleTransmission">
       <type>transmission_interface/SimpleTransmission</type>
-      <ros2_control name="GazeboSimSystem" type="system">
-        <hardware>
-          <plugin>gz_ros2_control/GazeboSimSystem</plugin>
-        </hardware>
-        <joint name="${name}_joint">
-          <hardwareInterface>hardware_interface/EffortJointInterface</hardwareInterface>
-        </joint>
-        <actuator name="${name}_motor">
-          <hardwareInterface>hardware_interface/EffortJointInterface</hardwareInterface>
-          <mechanicalReduction>1</mechanicalReduction>
-        </actuator>
-      </ros2_control>
+      <joint name="${name}_joint">
+        <hardwareInterface>hardware_interface/EffortJointInterface</hardwareInterface>
+      </joint>
+      <actuator name="${name}_motor">
+        <hardwareInterface>hardware_interface/EffortJointInterface</hardwareInterface>
+        <mechanicalReduction>1</mechanicalReduction>
+      </actuator>
     </transmission>
-  </xacro:macro>
-  <xacro:macro name="steering_hinge_transmission" params="name">
-    <transmission name="${name}_transmission" type="SimpleTransmission">
-      <type>transmission_interface/SimpleTransmission</type>
-      <ros2_control name="GazeboSimSystem" type="system">
-        <hardware>
-          <plugin>gz_ros2_control/GazeboSimSystem</plugin>
-        </hardware>
-        <joint name="${name}_joint">
-          <hardwareInterface>hardware_interface/EffortJointInterface</hardwareInterface>
-        </joint>
-        <actuator name="${name}_motor">
-          <hardwareInterface>hardware_interface/EffortJointInterface</hardwareInterface>
-          <mechanicalReduction>1</mechanicalReduction>
-        </actuator>
-      </ros2_control>
-    </transmission>
-  </xacro:macro>
+  </xacro:macro> -->
   <!-- Add chassis and it's inertia link -->
   <link name="$(arg robot_name)_base_link"/>
@@ -215,5 +212,5 @@
     <limit lower="-1.0" upper="1.0" effort="10" velocity="100" />
   </joint>
-  <xacro:steering_hinge_transmission name="$(arg robot_name)_left_steering_hinge" />
+  <!-- <xacro:steering_hinge_transmission name="$(arg robot_name)_left_steering_hinge" /> -->
   <!-- Add the right steering hinge with its joints and tranmissions -->
   <link name="$(arg robot_name)_right_steering_hinge">
@@ -233,5 +230,5 @@
     <limit lower="-1.0" upper="1.0" effort="10" velocity="100" />
   </joint>
-  <xacro:steering_hinge_transmission name="$(arg robot_name)_right_steering_hinge" />
+  <!-- <xacro:steering_hinge_transmission name="$(arg robot_name)_right_steering_hinge" /> -->
   <!-- Add the left front wheel with its joints and tranmissions -->
   <link name="$(arg robot_name)_left_front_wheel">
@@ -290,5 +287,5 @@
       <origin xyz="0 0 -0.018" rpy="0 0 0"/>
       <geometry>
-        <mesh filename="package://ros2_gazebo_sim/urdf/meshes/hokuyo.stl"/>
+        <mesh filename="model://urdf/meshes/hokuyo.stl"/>
         <material name="grey" />
       </geometry>
@@ -399,9 +396,12 @@
   <gazebo>
     <plugin filename="libgz_ros2_control-system.so" name="gz_ros2_control::GazeboSimROS2ControlPlugin">
-      <parameters>$(find gz_ros2_control_demos)/config/control.yaml</parameters>
+      <parameters>$(find ros2_gazebo_sim)/config/control.yaml</parameters>
     </plugin>
+    <ros>
+        <namespace>/$(arg robot_name)</namespace>
+      </ros>
   </gazebo>
   <!-- Odometry (cheap hack) -->
-  <gazebo>
+  <!-- <gazebo>
     <plugin name="p3d_base_controller" filename="libgazebo_ros_p3d.so">
       <alwaysOn>true</alwaysOn>
@@ -414,7 +414,7 @@
       <rpyOffsets>0 0 0</rpyOffsets>
     </plugin>
-  </gazebo>
+  </gazebo> -->
   <!-- hokuyo -->
-  <xacro:unless value="$(optenv DISABLE_GAZEBO_LASER false)">
+  <!-- <xacro:unless value="$(optenv DISABLE_GAZEBO_LASER false)">
     <gazebo reference="$(arg robot_name)_laser">
       <material>Gazebo/Grey</material>
@@ -448,13 +448,11 @@
       </sensor>
     </gazebo>
-  </xacro:unless>
+  </xacro:unless> -->
   <!-- camera object -->
-  <xacro:unless value="$(optenv DISABLE_GAZEBO_CAMERA false)">
+  <!-- <xacro:unless value="$(optenv DISABLE_GAZEBO_CAMERA false)">
     <gazebo reference="$(arg robot_name)_camera_link">
       <sensor type="camera" name="$(arg robot_name)_left_sensor">
         <update_rate>30.0</update_rate>
-        <!-- math.atan(320 / 687.8065795898438) * 2 -->
         <camera name="front_camera">
-          <!-- horizontal_fov>0.8709216071359963</horizontal_fov -->
           <horizontal_fov>1.74</horizontal_fov>
           <image>
@@ -480,5 +478,5 @@
           <cameraInfoTopicName>rgb/camera_info</cameraInfoTopicName>
           <frameName>$(arg robot_name)_camera_link</frameName>
-          <hackBaseline>0</hackBaseline><!-- set this to 0.12 for the second camera -->
+          <hackBaseline>0</hackBaseline>
           <distortionK1>0.0</distortionK1>
           <distortionK2>0.0</distortionK2>
@@ -489,5 +487,5 @@
       </sensor>
     </gazebo>
-  </xacro:unless>
+  </xacro:unless> -->
   <material name="black">
     <color rgba="0.0 0.0 0.0 1.0"/>

File: ros2_gazebo_sim/urdf/model.urdf (robot description, URDF)
Before this commit: robot virtual_robot, 13 links, 12 joints
Links:
- link car_1_chassis: geometry collision mesh filename=model://urdf/meshes/chassis.stl scale=0.000990 0.0009375 0.0009375; visual mesh filename=model://urdf/meshes/chassis.stl scale=0.000990 0.0009375 0.0009375
- link car_1_laser: geometry collision box size=0.1 0.1 0.1; visual mesh filename=model://urdf/meshes/hokuyo.stl
- link car_1_left_front_wheel: geometry collision cylinder length=0.045 radius=0.05; visual mesh filename=model://urdf/meshes/left_wheel.stl
- link car_1_left_rear_wheel: geometry collision cylinder length=0.045 radius=0.05; visual mesh filename=model://urdf/meshes/left_wheel.stl
- link car_1_left_steering_hinge: geometry visual mesh filename=model://urdf/meshes/hinge.stl
- link car_1_right_front_wheel: geometry collision cylinder length=0.045 radius=0.05; visual mesh filename=model://urdf/meshes/right_wheel.stl
- link car_1_right_rear_wheel: geometry collision cylinder length=0.045 radius=0.05; visual mesh filename=model://urdf/meshes/right_wheel.stl
- link car_1_right_steering_hinge: geometry visual mesh filename=model://urdf/meshes/hinge.stl

Commit message: STEERING IS WORKING

File: ros2_gazebo_sim/urdf/macros.xacro (robot description, xacro)
@@ -102,29 +102,21 @@
       </hardware>
       <joint name="${name}_joint">
+        <command_interface name="velocity" />
+        <state_interface name="velocity" />
+        <state_interface name="position" />
       </joint>
     </ros2_control>
-    <!-- <transmission name="${name}_transmission" type="SimpleTransmission">
-      <type>transmission_interface/SimpleTransmission</type>
+  </xacro:macro>
+  <xacro:macro name="steering_hinge_transmission" params="name">
+    <ros2_control name="${name}_transmission" type="actuator">
+      <hardware>
+        <plugin>gz_ros2_control/GazeboSimSystem</plugin>
+      </hardware>
       <joint name="${name}_joint">
-        <hardwareInterface>hardware_interface/EffortJointInterface</hardwareInterface>
+        <command_interface name="position" />
+        <state_interface name="position" />
       </joint>
-      <actuator name="${name}_motor">
-        <hardwareInterface>hardware_interface/EffortJointInterface</hardwareInterface>
-        <mechanicalReduction>1</mechanicalReduction>
-      </actuator>
-    </transmission> -->
-  </xacro:macro>
-  <!-- <xacro:macro name="steering_hinge_transmission" params="name">
-    <transmission name="${name}_transmission" type="SimpleTransmission">
-      <type>transmission_interface/SimpleTransmission</type>
-      <joint name="${name}_joint">
-        <hardwareInterface>hardware_interface/EffortJointInterface</hardwareInterface>
-      </joint>
-      <actuator name="${name}_motor">
-        <hardwareInterface>hardware_interface/EffortJointInterface</hardwareInterface>
-        <mechanicalReduction>1</mechanicalReduction>
-      </actuator>
-    </transmission>
-  </xacro:macro> -->
+    </ros2_control>
+  </xacro:macro>
   <!-- Add chassis and it's inertia link -->
   <link name="$(arg robot_name)_base_link"/>
@@ -212,5 +204,5 @@
     <limit lower="-1.0" upper="1.0" effort="10" velocity="100" />
   </joint>
-  <!-- <xacro:steering_hinge_transmission name="$(arg robot_name)_left_steering_hinge" /> -->
+  <xacro:steering_hinge_transmission name="$(arg robot_name)_left_steering_hinge" />
   <!-- Add the right steering hinge with its joints and tranmissions -->
   <link name="$(arg robot_name)_right_steering_hinge">
@@ -230,5 +222,5 @@
     <limit lower="-1.0" upper="1.0" effort="10" velocity="100" />
   </joint>
-  <!-- <xacro:steering_hinge_transmission name="$(arg robot_name)_right_steering_hinge" /> -->
+  <xacro:steering_hinge_transmission name="$(arg robot_name)_right_steering_hinge" />
   <!-- Add the left front wheel with its joints and tranmissions -->
   <link name="$(arg robot_name)_left_front_wheel">
