Commit message: imu working alongside all other sensors plus movement

File: ros2_gazebo_sim/urdf/macros.xacro (robot description, xacro)
@@ -5,4 +5,11 @@
   <xacro:arg name="robot_skin" default="Blue" />
   <!-- inertial parameter macros -->
+  <xacro:macro name="box_inertia" params="m w h d">
+    <inertial>
+      <origin xyz="0 0 0" rpy="${pi/2} 0 ${pi/2}"/>
+      <mass value="${m}"/>
+      <inertia ixx="${(m/12) * (h*h + d*d)}" ixy="0.0" ixz="0.0" iyy="${(m/12) * (w*w + d*d)}" iyz="0.0" izz="${(m/12) * (w*w + h*h)}"/>
+    </inertial>
+  </xacro:macro>
   <xacro:macro name="chassis_inertial_params">
     <origin xyz="0.1477 0 0" rpy="0 0 0" />
@@ -145,4 +152,23 @@
     <child link="$(arg robot_name)_chassis_inertia" />
   </joint>
+  <!-- Add the imu sensor -->
+  <link name="$(arg robot_name)_imu_link">
+    <visual>
+      <geometry>
+        <box size="0.1 0.1 0.1"/>
+      </geometry>
+    </visual>
+    <collision>
+      <geometry>
+        <box size="0.1 0.1 0.1"/>
+      </geometry>
+    </collision>
+    <xacro:box_inertia m="0.1" w="0.1" d="0.1" h="0.1"/>
+  </link>
+  <joint name="$(arg robot_name)_imu_joint" type="fixed">
+    <parent link="$(arg robot_name)_chassis"/>
+    <child link="$(arg robot_name)_imu_link"/>
+    <origin xyz="0 0 0.01"/>
+  </joint>
   <!-- Add the left rear wheel with its joints and tranmissions -->
   <link name="$(arg robot_name)_left_rear_wheel">
@@ -388,9 +414,71 @@
   <gazebo>
     <plugin filename="libgz_ros2_control-system.so" name="gz_ros2_control::GazeboSimROS2ControlPlugin">
-      <parameters>$(find ros2_gazebo_sim)/config/control.yaml</parameters>
+      <parameters>$(find ros2_gazebo_sim)/config/control_odom.yaml</parameters>
     </plugin>
     <ros>
         <namespace>/$(arg robot_name)</namespace>
       </ros>
+  </gazebo>
+  <!-- IMU -->
+  <gazebo reference="$(arg robot_name)_imu_link">
+    <sensor name="$(arg robot_name)_imu_sensor" type="imu">
+      <always_on>true</always_on>
+      <update_rate>1</update_rate>
+      <topic>/$(arg robot_name)/imu</topic>
+      <imu>
+        <angular_velocity>
+          <x>
+            <noise type="gaussian">
+              <mean>0.0</mean>
+              <stddev>2e-4</stddev>
+              <bias_mean>0.0000075</bias_mean>
+              <bias_stddev>0.0000008</bias_stddev>
+            </noise>
+          </x>
+          <y>
+            <noise type="gaussian">
+              <mean>0.0</mean>
+              <stddev>2e-4</stddev>
+              <bias_mean>0.0000075</bias_mean>
+              <bias_stddev>0.0000008</bias_stddev>
+            </noise>
+          </y>
+          <z>
+            <noise type="gaussian">
+              <mean>0.0</mean>
+              <stddev>2e-4</stddev>
+              <bias_mean>0.0000075</bias_mean>
+              <bias_stddev>0.0000008</bias_stddev>
+            </noise>
+          </z>
+        </angular_velocity>
+        <linear_acceleration>
+          <x>
+            <noise type="gaussian">
+              <mean>0.0</mean>
+              <stddev>1.7e-2</stddev>
+              <bias_mean>0.1</bias_mean>
+              <bias_stddev>0.001</bias_stddev>
+            </noise>
+          </x>
+          <y>
+            <noise type="gaussian">
+              <mean>0.0</mean>
+              <stddev>1.7e-2</stddev>
+              <bias_mean>0.1</bias_mean>
+              <bias_stddev>0.001</bias_stddev>
+            </noise>
+          </y>
+          <z>
+            <noise type="gaussian">
+              <mean>0.0</mean>
+              <stddev>1.7e-2</stddev>
+              <bias_mean>0.1</bias_mean>
+              <bias_stddev>0.001</bias_stddev>
+            </noise>
+          </z>
+        </linear_acceleration>
+      </imu>
+    </sensor>
   </gazebo>
   <!-- hokuyo -->
@@ -426,34 +514,4 @@
     </gazebo>
   </xacro:unless>
-  <!-- camera object -->
-  <xacro:unless value="$(optenv DISABLE_GAZEBO_CAMERA false)">
-    <gazebo reference="$(arg robot_name)_camera_link">
-      <sensor type="camera" name="$(arg robot_name)_left_sensor">
-        <topic>/$(arg robot_name)/camera/image_raw</topic>
-        <update_rate>30.0</update_rate>
-        <always_on>true</always_on>
-        <visualize>true</visualize>
-        <gz_frame_id>$(arg robot_name)_camera_link</gz_frame_id>
-        <camera name="front_camera">
-          <camera_info_topic>/$(arg robot_name)/camera_info</camera_info_topic>
-          <horizontal_fov>1.74</horizontal_fov>
-          <image>
-            <width>1920</width>
-            <height>1080</height>
-            <format>B8G8R8</format>
-          </image>
-          <clip>
-            <near>0.02</near>
-            <far>300</far>
-          </clip>
-          <noise>
-            <type>gaussian</type>
-            <mean>0.0</mean>
-            <stddev>0.007</stddev>
-          </noise>
-        </camera>
-      </sensor>
-    </gazebo>
-  </xacro:unless>
   <material name="black">
     <color rgba="0.0 0.0 0.0 1.0"/>

File: ros2_gazebo_sim/urdf/model.urdf (robot description, URDF)
Before this commit: robot virtual_robot, 14 links, 13 joints
Links:
- removed link base_link
- removed link camera_link
- removed link chassis
- removed link chassis_inertia
- removed link imu_link
- removed link laser
- removed link left_front_wheel
- removed link left_rear_wheel
- removed link left_steering_hinge
- removed link link
- removed link right_front_wheel
- removed link right_link
- removed link right_rear_wheel
- removed link right_steering_hinge
- added link car_1_base_link
- added link car_1_camera_link, mass 1e-5
- added link car_1_chassis; collision mesh filename=model://urdf/meshes/chassis.stl scale=0.000990 0.0009375 0.0009375; visual mesh filename=model://urdf/meshes/chassis.stl scale=0.000990 0.0009375 0.0009375
- added link car_1_chassis_inertia, mass 4.0
- added link car_1_imu_link, mass 0.1; collision box size=0.1 0.1 0.1; visual box size=0.1 0.1 0.1
- added link car_1_laser, mass 0.130; collision box size=0.1 0.1 0.1; visual mesh filename=model://urdf/meshes/hokuyo.stl
- added link car_1_left_front_wheel, mass 0.34055; collision cylinder length=0.045 radius=0.05; visual mesh filename=model://urdf/meshes/left_wheel.stl
- added link car_1_left_rear_wheel, mass 0.34055; collision cylinder length=0.045 radius=0.05; visual mesh filename=model://urdf/meshes/left_wheel.stl
- added link car_1_left_steering_hinge, mass 0.100; visual mesh filename=model://urdf/meshes/hinge.stl
- added link car_1_link, mass 1e-5; collision box size=0.033 0.175 0.030; visual box size=0.033 0.175 0.030
- added link car_1_right_front_wheel, mass 0.34055; collision cylinder length=0.045 radius=0.05; visual mesh filename=model://urdf/meshes/right_wheel.stl
- added link car_1_right_link, mass 1e-5
- added link car_1_right_rear_wheel, mass 0.34055; collision cylinder length=0.045 radius=0.05; visual mesh filename=model://urdf/meshes/right_wheel.stl
- added link car_1_right_steering_hinge, mass 0.100; visual mesh filename=model://urdf/meshes/hinge.stl
Joints:
- removed joint base_link_joint
- removed joint chassis_inertia_joint
- removed joint hokuyo_joint
- removed joint imu_joint
- removed joint joint
- removed joint left_front_wheel_joint
- removed joint left_joint
- removed joint left_rear_wheel_joint
- removed joint left_steering_hinge_joint
- removed joint right_front_wheel_joint
- removed joint right_joint
- removed joint right_rear_wheel_joint
- removed joint right_steering_hinge_joint
- added joint car_1_base_link_joint: type fixed, parent car_1_base_link, child car_1_chassis, origin xyz=0 0 0.05 rpy=0 0 0
- added joint car_1_chassis_inertia_joint: type fixed, parent car_1_chassis, child car_1_chassis_inertia, origin xyz=0 0 0 rpy=0 0 0
- added joint car_1_hokuyo_joint: type fixed, parent car_1_chassis, child car_1_laser, origin xyz=0.125 0.0 0.173 rpy=0 0 0, axis 0 0 1
- added joint car_1_imu_joint: type fixed, parent car_1_chassis, child car_1_imu_link, origin xyz=0 0 0.01
- added joint car_1_joint: type fixed, parent car_1_chassis, child car_1_link, origin xyz=0.390 0 0.025 rpy=0 0 0, axis 0 0 1
- added joint car_1_left_front_wheel_joint: type continuous, parent car_1_left_steering_hinge, child car_1_left_front_wheel, origin xyz=0 0 0 rpy=1.5708 0 0, axis 0 0 -1, limit effort=10 velocity=100
- added joint car_1_left_joint: type fixed, parent car_1_link, child car_1_camera_link, origin xyz=-2.5 0 1.75 rpy=0 .57 0, axis 0 0 1
- added joint car_1_left_rear_wheel_joint: type continuous, parent car_1_chassis, child car_1_left_rear_wheel, origin xyz=0 0.1 0 rpy=1.5708 0 0, axis 0 0 -1, limit effort=10 velocity=100
- added joint car_1_left_steering_hinge_joint: type revolute, parent car_1_chassis, child car_1_left_steering_hinge, origin xyz=0.325 0.1 0 rpy=0 1.5708 0, axis -1 0 0, limit lower=-1.0 upper=1.0 effort=10 velocity=100
- added joint car_1_right_front_wheel_joint: type continuous, parent car_1_right_steering_hinge, child car_1_right_front_wheel, origin xyz=0 0 0 rpy=1.5708 0 0, axis 0 0 -1, limit effort=10 velocity=100
- added joint car_1_right_joint: type fixed, parent car_1_link, child car_1_right_link, origin xyz=0 -0.06 0.025 rpy=0 0 0, axis 0 0 1
- added joint car_1_right_rear_wheel_joint: type continuous, parent car_1_chassis, child car_1_right_rear_wheel, origin xyz=0 -0.1 0 rpy=1.5708 0 0, axis 0 0 -1, limit effort=10 velocity=100
- added joint car_1_right_steering_hinge_joint: type revolute, parent car_1_chassis, child car_1_right_steering_hinge, origin xyz=0.325 -0.1 0 rpy=0 1.5708 0, axis -1 0 0, limit lower=-1.0 upper=1.0 effort=10 velocity=100

Commit message: added EKF to fuse imu and odom data

File: ros2_gazebo_sim/urdf/macros.xacro (robot description, xacro)
@@ -127,5 +127,6 @@
   </xacro:macro>
   <!-- Add chassis and it's inertia link -->
-  <link name="$(arg robot_name)_base_link"/>
+  <!-- <link name="$(arg robot_name)_base_link"/> -->
+  <link name="base_link"/>
   <link name="$(arg robot_name)_chassis">
     <visual>
@@ -139,5 +140,5 @@
   <joint name="$(arg robot_name)_base_link_joint" type="fixed">
     <origin xyz="0 0 0.05" rpy="0 0 0" />
-    <parent link="$(arg robot_name)_base_link" />
+    <parent link="base_link" />
     <child link="$(arg robot_name)_chassis" />
   </joint>

File: ros2_gazebo_sim/urdf/model.urdf (robot description, URDF)
Before this commit: robot virtual_robot, 14 links, 13 joints
Links:
- removed link car_1_base_link
- added link base_link
Joints:
- joint car_1_base_link_joint: parent car_1_base_link -> base_link

Commit message: saved chassis z at 0.05 like it originally was

File: ros2_gazebo_sim/urdf/macros.xacro (robot description, xacro)
@@ -170,5 +170,5 @@
     <parent link="$(arg robot_name)_chassis"/>
     <child link="$(arg robot_name)_imu_link"/>
-    <origin xyz="0 0 0.01"/>
+    <origin xyz="0 0 0.05"/>
   </joint>
   <!-- Add the left rear wheel with its joints and tranmissions -->

Commit message: added node to broadcast poses for exploring the map before loop closure is achieved

File: ros2_gazebo_sim/urdf/macros.xacro (robot description, xacro)
@@ -137,4 +137,7 @@
       <xacro:chassis_geometry />
     </collision>
+    <inertial>
+      <xacro:chassis_inertial_params />
+    </inertial>
   </link>
   <joint name="$(arg robot_name)_base_link_joint" type="fixed">
@@ -143,14 +146,14 @@
     <child link="$(arg robot_name)_chassis" />
   </joint>
-  <link name="$(arg robot_name)_chassis_inertia">
+  <!-- <link name="$(arg robot_name)_chassis_inertia">
     <inertial>
       <xacro:chassis_inertial_params />
     </inertial>
-  </link>
-  <joint name="$(arg robot_name)_chassis_inertia_joint" type="fixed">
+  </link> -->
+  <!-- <joint name="$(arg robot_name)_chassis_inertia_joint" type="fixed">
     <origin xyz="0 0 0" rpy="0 0 0" />
     <parent link="$(arg robot_name)_chassis" />
     <child link="$(arg robot_name)_chassis_inertia" />
-  </joint>
+  </joint> -->
   <!-- Add the imu sensor -->
   <link name="$(arg robot_name)_imu_link">
